File: pcb/krunchcard.kicad_pcb (KiCad board)
At the start: 2 copper layers, 86 x 54 mm, 42 parts, among them U1 NT3H2111W0FTTJ

Commit message: updated copper pour around antenna, reworked infos
Other:
- board text added: "github: curl api.github.com/user/75719839 web: krunch.hackclub.app"
- board text removed: "web: krunch.hackclub.app github id: 757198399/RadioactivePotato"
Changed lines of the file:
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@@
 			(outputformat 1)
 			(mirror no)
-			(drillshape 1)
+			(drillshape 0)
 			(scaleselection 1)
-			(outputdirectory "")
+			(outputdirectory "C:/Users/root/Downloads/GERBER/")
 		)
 	)
@@
 			(at 0 4.2 0)
 			(layer "F.Fab")
+			(hide yes)
 			(effects
 				(font
@@
 			(at 0 4.7244 0)
 			(layer "B.SilkS")
+			(hide yes)
 			(effects
 				(font
@@
 		(layer "Edge.Cuts")
 	)
-	(gr_text "web: krunch.hackclub.app\ngithub id: 757198399/RadioactivePotato"
-		(at 114.5 86.5 0)
+	(gr_text "github:\ncurl api.github.com/user/75719839\n\nweb:\nkrunch.hackclub.app"
+		(at 138.6 90.1 0)
 		(layer "F.SilkS")
 		(effects
 			(font
-				(size 1.6256 1.6256)
-				(thickness 0.2032)
+				(size 1.5 1.5)
+				(thickness 0.2)
 			)
-			(justify left top)
+			(justify top)
 		)
 	)
@@
 		(layer "F.Cu")
 		(hatch edge 0.5)
-		(priority 6)
-		(connect_pads
-			(clearance 0.5)
-		)
-		(min_thickness 0.25)
-		(filled_areas_thickness no)
-		(fill yes
-			(thermal_gap 0.5)
-			(thermal_bridge_width 0.5)
-			(island_removal_mode 1)
-			(island_area_min 10)
-		)
-		(polygon
-			(pts
-				(xy 161.75 114) (xy 161 114.75) (xy 161 118.5) (xy 163.25 118.5) (xy 163.25 122.5) (xy 166 122.5)
-				(xy 166 114)
-			)
-		)
-	)
-	(zone
-		(net 0)
-		(net_name "")
-		(layer "F.Cu")
-		(hatch edge 0.5)
 		(priority 8)
 		(connect_pads
@@
 		(layer "F.Cu")
 		(hatch edge 0.5)
-		(priority 7)
+		(priority 8)
 		(connect_pads
 			(clearance 0.5)
@@
 		(polygon
 			(pts
-				(xy 162 108.25) (xy 162 112.75) (xy 165.75 112.75) (xy 166.205 112.386) (xy 166.205 108.25)
+				(xy 165.5 122.519) (xy 163.25 122.519) (xy 163.25 118.5) (xy 161.75 118.5) (xy 161.75 108) (xy 165.5 108)
 			)
 		)
@@
 		(polygon
 			(pts
-				(xy 107.75 77.5) (xy 166.71014 77.5) (xy 166.51014 135) (xy 107.75 135)
-			)
-		)
-	)
-	(zone
-		(net 0)
-		(net_name "")
-		(layers "F.Cu" "B.Cu")
-		(hatch edge 0.5)
-		(priority 2)
-		(connect_pads
-			(clearance 0.5)
-		)
-		(min_thickness 0.25)
-		(filled_areas_thickness no)
-		(fill yes
-			(thermal_gap 0.5)
-			(thermal_bridge_width 0.5)
-			(island_removal_mode 1)
-			(island_area_min 10)
-		)
-		(polygon
-			(pts
-				(xy 198 77.5) (xy 194.5 77.5) (xy 194.5 135) (xy 198 135)
-			)
-		)
-	)
-	(zone
-		(net 0)
-		(net_name "")
-		(layers "F.Cu" "B.Cu")
-		(hatch edge 0.5)
-		(priority 1)
-		(connect_pads
-			(clearance 0.5)
-		)
-		(min_thickness 0.25)
-		(filled_areas_thickness no)
-		(fill yes
-			(thermal_gap 0.5)
-			(thermal_bridge_width 0.5)
-			(island_removal_mode 1)
-			(island_area_min 10)
-		)
-		(polygon
-			(pts
-				(xy 194.75 135) (xy 194.75 132) (xy 166.25 132) (xy 166.25 135)
-			)
-		)
-	)
-	(zone
-		(net 0)
-		(net_name "")
-		(layers "F.Cu" "B.Cu")
-		(hatch edge 0.5)
-		(priority 3)
-		(connect_pads
-			(clearance 0.5)
-		)
-		(min_thickness 0.25)
-		(filled_areas_thickness no)
-		(fill yes
-			(thermal_gap 0.5)
-			(thermal_bridge_width 0.5)
-			(island_removal_mode 1)
-			(island_area_min 10)
-		)
-		(polygon
-			(pts
-				(xy 195 81.5) (xy 166.25 81.5) (xy 166.25 77.5) (xy 195 77.5)
+				(xy 107.75 77.5) (xy 165.703702 77.5) (xy 165.503702 135) (xy 107.75 135)
 			)
 		)
@@
 		(polygon
 			(pts
-				(xy 166.6 77.5) (xy 166.6 135) (xy 107.75 135) (xy 107.75 77.5)
+				(xy 165.703702 77.5) (xy 165.503702 135) (xy 107.75 135) (xy 107.75 77.5)
 			)
 		)
